Commit message: Created gz to ros bridge

File: diff_drive/urdf/ddrive.gazebo.xacro (robot description, xacro)
@@ -18,6 +18,6 @@
           filename="libgz-sim-diff-drive-system.so"
           name="gz::sim::systems::DiffDrive">
-          <left_joint>left_wheel_joint</left_joint>
-          <right_joint>right_wheel_joint</right_joint>
+          <left_joint>wheel_left_joint</left_joint>
+          <right_joint>wheel_right_joint</right_joint>
           <wheel_separation>1.25</wheel_separation>
           <wheel_radius>0.3</wheel_radius>
@@ -29,12 +29,6 @@
             filename="libgz-sim-joint-state-publisher-system.so"
             name="gz::sim::systems::JointStatePublisher">
-            </plugin>
-       </gazebo>
-    <plugin filename="gz-sim-joint-state-publisher-system" name="gz::sim::systems::JointStatePublisher">
-        <update_rate>20</update_rate>
-        <topic>joint_states</topic>
-        <joint_name>wheel1_joint</joint_name>
-        <joint_name>wheel2_joint</joint_name>
-    </plugin>
+        </plugin>
+    </gazebo>
 </gazebo>
 </robot>

File: diff_drive/urdf/ddrive.urdf.xacro (robot description, xacro)
@@ -1,4 +1,4 @@
 <?xml version="1.0"?>
-<robot name="my_robot" xmlns:xacro="http://www.ros.org/wiki/xacro">
+<robot name="diff_drive" xmlns:xacro="http://www.ros.org/wiki/xacro">
     <xacro:property name="pi_const" value="3.14159265" />
     <!-- Body dimensions -->
@@ -73,4 +73,7 @@
                 <box size="${a} ${c} ${b}" />
             </geometry>
+            <material name="red">
+                <color rgba="1 0 0 1"/>
+              </material>
         </visual>
         <collision>
@@ -87,4 +90,7 @@
                 <cylinder radius="${r}" length="${d}" />
             </geometry>
+            <material name="red">
+                <color rgba="1 1 0 1"/>
+              </material>
         </visual>
         <collision>
@@ -101,4 +107,7 @@
                 <cylinder radius="${r}" length="${d}" />
             </geometry>
+            <material name="red">
+                <color rgba="1 1 0 1"/>
+              </material>
         </visual>
         <collision>
@@ -115,4 +124,7 @@
                 <sphere radius="${r/2}" />
             </geometry>
+            <material name="red">
+                <color rgba="1 0 1 1"/>
+              </material>
         </visual>
         <collision>
@@ -129,4 +141,7 @@
                 <sphere radius="${r/2}" />
             </geometry>
+            <material name="red">
+                <color rgba="1 0 1 1"/>
+              </material>
         </visual>
         <collision>

Commit message: Fix gazebo publishers

File: diff_drive/urdf/ddrive.gazebo.xacro (robot description, xacro)
@@ -1,34 +1,26 @@
 <?xml version="1.0"?>
-<robot>
-<gazebo reference="base_link">
-    <material>Gazebo/Red</material>
-</gazebo>
-<gazebo reference="wheel1_link">
-    <material>Gazebo/Yellow</material>
-</gazebo>
-<gazebo reference="wheel2_link">
-    <material>Gazebo/Yellow</material>
-</gazebo>
-<gazebo reference="caster_link">
-    <material>Gazebo/Blue</material>
-</gazebo>
-<gazebo>
+<robot xmlns:xacro="http://www.ros.org/wiki/xacro">
     <gazebo>
         <plugin
-          filename="libgz-sim-diff-drive-system.so"
-          name="gz::sim::systems::DiffDrive">
-          <left_joint>wheel_left_joint</left_joint>
-          <right_joint>wheel_right_joint</right_joint>
-          <wheel_separation>1.25</wheel_separation>
-          <wheel_radius>0.3</wheel_radius>
-          <odom_publish_frequency>50</odom_publish_frequency>
-          <frame_id>odom</frame_id>
-          <child_frame_id>base_link</child_frame_id>
+            filename="gz-sim-diff-drive-system"
+            name="gz::sim::systems::DiffDrive">
+            <left_joint>wheel_left_joint</left_joint>
+            <right_joint>wheel_right_joint</right_joint>
+            <wheel_separation>1.25</wheel_separation>
+            <wheel_radius>0.3</wheel_radius>
+            <odom_publish_frequency>50</odom_publish_frequency>
+            <frame_id>odom</frame_id>
+            <child_frame_id>base_link</child_frame_id>
         </plugin>
         <plugin
-            filename="libgz-sim-joint-state-publisher-system.so"
+            filename="sim-joint-state-publisher-system"
             name="gz::sim::systems::JointStatePublisher">
         </plugin>
+        <plugin filename="libgz-sim-joint-state-publisher-system"
+            name="gz::sim::systems::JointStatePublisher">
+            <topic>/joint_states</topic>
+            <joint_name>wheel_left_joint</joint_name>
+            <joint_name>wheel_right_joint</joint_name>
+        </plugin>
     </gazebo>
-</gazebo>
 </robot>

File: diff_drive/urdf/ddrive.urdf.xacro (robot description, xacro)
@@ -182,4 +182,4 @@
         <origin xyz="${s4 - 0.1} 0 -${s1}" rpy="0 0 0" />
     </joint>
-    <include file="$(find diff_drive)/urdf/ddrive.gazebo.xacro" />
+    <xacro:include filename="/home/david/cls/_ME495/src/hw3/src/diff_drive/urdf/ddrive.gazebo.xacro"/>
 </robot>

Commit message: Added gz bridge

File: diff_drive/urdf/ddrive.gazebo.xacro (robot description, xacro)
@@ -12,14 +12,8 @@
             <frame_id>odom</frame_id>
             <child_frame_id>base_link</child_frame_id>
+            <topic>/cmd_vel</topic>
         </plugin>
-        <plugin
-            filename="sim-joint-state-publisher-system"
+        <plugin filename="libgz-sim-joint-state-publisher-system.so"
             name="gz::sim::systems::JointStatePublisher">
-        </plugin>
-        <plugin filename="libgz-sim-joint-state-publisher-system"
-            name="gz::sim::systems::JointStatePublisher">
-            <topic>/joint_states</topic>
-            <joint_name>wheel_left_joint</joint_name>
-            <joint_name>wheel_right_joint</joint_name>
         </plugin>
     </gazebo>

File: diff_drive/urdf/ddrive.urdf.xacro (robot description, xacro)
@@ -15,7 +15,7 @@
     <xacro:property name="s4" value="${a/2}" />
     <!-- Robot body mass and inertia properties -->
-    <xacro:property name="m1" value="5.0" /> <!-- Body mass -->
-    <xacro:property name="m2" value="0.5" /> <!-- Wheel mass -->
-    <xacro:property name="m3" value="0.2" /> <!-- Caster mass -->
+    <xacro:property name="m1" value="1.0" /> <!-- Body mass -->
+    <xacro:property name="m2" value="10.0" /> <!-- Wheel mass -->
+    <xacro:property name="m3" value="1.0" /> <!-- Caster mass -->
     <xacro:macro name="inertia_body">
         <inertial>
@@ -33,5 +33,5 @@
     <xacro:macro name="inertia_wheel">
         <inertial>
-            <mass value="2.0" />
+            <mass value="${m2}" />
             <inertia
                 ixx="0.145833"
@@ -46,5 +46,5 @@
     <xacro:macro name="inertia_caster">
         <inertial>
-            <mass value="0.1" />
+            <mass value="${m3}" />
             <inertia
                 ixx="0.0001"
@@ -57,14 +57,4 @@
         </inertial>
     </xacro:macro>
-    <link name="base_footprint">
-        <visual>
-            <geometry>
-                <box size="0.01 0.01 0.01" /> <!-- A small box to define the footprint -->
-            </geometry>
-            <material name="Grey">
-                <color rgba="0.5 0.5 0.5 1.0" />
-            </material>
-        </visual>
-    </link>
     <!-- Main body -->
     <link name="base_link">
@@ -73,5 +63,5 @@
                 <box size="${a} ${c} ${b}" />
             </geometry>
-            <material name="red">
+            <material name="blue">
                 <color rgba="1 0 0 1"/>
               </material>
@@ -82,5 +72,4 @@
             </geometry>
         </collision>
-        <xacro:inertia_body />
     </link>
     <!-- Rear left wheel -->
@@ -124,5 +113,5 @@
                 <sphere radius="${r/2}" />
             </geometry>
-            <material name="red">
+            <material name="yellow">
                 <color rgba="1 0 1 1"/>
               </material>
@@ -141,5 +130,5 @@
                 <sphere radius="${r/2}" />
             </geometry>
-            <material name="red">
+            <material name="yellow">
                 <color rgba="1 0 1 1"/>
               </material>
@@ -152,9 +141,4 @@
         <xacro:inertia_caster />
     </link>
-    <!-- Joints -->
-    <joint name="base_fixed_joint" type="fixed">
-        <parent link="base_footprint" />
-        <child link="base_link" />
-    </joint>
     <!-- Rear wheels joints -->
     <joint name="wheel_left_joint" type="continuous">
