Commit message: Robot flips

File: diff_drive/urdf/ddrive.urdf.xacro (robot description, xacro)
@@ -8,4 +8,5 @@
     <!-- Wheel and caster dimensions -->
     <xacro:property name="r" value="0.1" /> <!-- Radius for wheels and casters -->
+    <xacro:property name="wheel_radius" value="0.3" /> <!-- Radius for wheels and casters -->
     <xacro:property name="d" value="0.1" /> <!-- Thickness for wheels -->
     <!-- Positions -->
@@ -14,4 +15,5 @@
     <xacro:property name="s3" value="${c/2}" />
     <xacro:property name="s4" value="${a/2}" />
+    <xacro:property name="s5" value="${b/24}" />
     <!-- Robot body mass and inertia properties -->
     <xacro:property name="m1" value="1.0" /> <!-- Body mass -->
@@ -77,5 +79,5 @@
         <visual>
             <geometry>
-                <cylinder radius="${r}" length="${d}" />
+                <cylinder radius="${wheel_radius}" length="${d}" />
             </geometry>
             <material name="red">
@@ -85,5 +87,5 @@
         <collision>
             <geometry>
-                <cylinder radius="${r}" length="${d}" />
+                <cylinder radius="${wheel_radius}" length="${d}" />
             </geometry>
         </collision>
@@ -94,5 +96,5 @@
         <visual>
             <geometry>
-                <cylinder radius="${r}" length="${d}" />
+                <cylinder radius="${wheel_radius}" length="${d}" />
             </geometry>
             <material name="red">
@@ -102,5 +104,5 @@
         <collision>
             <geometry>
-                <cylinder radius="${r}" length="${d}" />
+                <cylinder radius="${wheel_radius}" length="${d}" />
             </geometry>
         </collision>
@@ -145,5 +147,5 @@
         <parent link="base_link" />
         <child link="wheel_left_link" />
-        <origin xyz="${-s4} ${s3} -${s1}" rpy="1.57 0 0" />
+        <origin xyz="${-s4} ${s3} -${s5}" rpy="1.57 0 0" />
         <axis xyz="0 0 1" />
     </joint>
@@ -151,5 +153,5 @@
         <parent link="base_link" />
         <child link="wheel_right_link" />
-        <origin xyz="${-s4} -${s3} -${s1}" rpy="1.57 0 0" />
+        <origin xyz="${-s4} -${s3} -${s5}" rpy="1.57 0 0" />
         <axis xyz="0 0 1" />
     </joint>

Commit message: Parameterize

File: diff_drive/urdf/ddrive.urdf.xacro (robot description, xacro)
@@ -1,13 +1,23 @@
 <?xml version="1.0"?>
 <robot name="diff_drive" xmlns:xacro="http://www.ros.org/wiki/xacro">
-    <xacro:property name="pi_const" value="3.14159265" />
+    <xacro:property name="yaml_file" value="$(find diff_drive)/params.yaml"/>
+    <xacro:property name="props" value="${xacro.load_yaml(yaml_file)['/**']['ros__parameters']}"/>
+    <xacro:property name="wheel_props" value="${props['wheel_dimensions']}"/>
+    <xacro:property name="caster_props" value="${props['caster_dimensions']}"/>
+    <xacro:property name="mass_props" value="${props['masses']}"/>
+    <xacro:property name="robot_props" value="${props['robot_dimensions']}"/>
     <!-- Body dimensions -->
-    <xacro:property name="a" value="1.0" /> <!-- Length -->
-    <xacro:property name="b" value="0.3" /> <!-- Height -->
-    <xacro:property name="c" value="0.6" /> <!-- Width -->
-    <!-- Wheel and caster dimensions -->
-    <xacro:property name="r" value="0.1" /> <!-- Radius for wheels and casters -->
-    <xacro:property name="wheel_radius" value="0.3" /> <!-- Radius for wheels and casters -->
-    <xacro:property name="d" value="0.1" /> <!-- Thickness for wheels -->
+    <xacro:property name="a" value="${robot_props['body_length']}" />
+    <xacro:property name="b" value="${robot_props['body_height']}" />
+    <xacro:property name="c" value="${robot_props['body_width']}" />
+    <!-- Wheel dimensions -->
+    <xacro:property name="wheel_radius" value="${wheel_props['wheel_radius']}" />
+    <xacro:property name="d" value="${wheel_props['wheel_thickness']}" />
+    <!-- Caster dimensions -->
+    <xacro:property name="r" value="${caster_props['caster_radius']}" />
+    <!-- Masses -->
+    <xacro:property name="m1" value="${mass_props['body_mass']}" />
+    <xacro:property name="m2" value="${mass_props['wheel_mass']}" />
+    <xacro:property name="m3" value="${mass_props['caster_mass']}" />
     <!-- Positions -->
     <xacro:property name="s1" value="${b/2}" />
@@ -16,8 +26,4 @@
     <xacro:property name="s4" value="${a/2}" />
     <xacro:property name="s5" value="${b/24}" />
-    <!-- Robot body mass and inertia properties -->
-    <xacro:property name="m1" value="1.0" /> <!-- Body mass -->
-    <xacro:property name="m2" value="10.0" /> <!-- Wheel mass -->
-    <xacro:property name="m3" value="1.0" /> <!-- Caster mass -->
     <xacro:macro name="inertia_body">
         <inertial>
@@ -168,4 +174,4 @@
         <origin xyz="${s4 - 0.1} 0 -${s1}" rpy="0 0 0" />
     </joint>
-    <xacro:include filename="/home/david/cls/_ME495/src/hw3/src/diff_drive/urdf/ddrive.gazebo.xacro"/>
+    <xacro:include filename="$(find diff_drive)/ddrive.gazebo.xacro"/>
 </robot>
